Commit message: Changed the steering joint placement at the center of each tire

File: urdf/catvehicle.xacro (robot description, xacro)
@@ -76,5 +76,5 @@
     <xacro:property name="tyre_length" value="0.2336291492"/>
     <xacro:property name="tyre_radius" value="0.3671951254"/>
-    <xacro:property name="tyre_mass" value="100"/>
+    <xacro:property name="tyre_mass" value="20"/>
     <!--xacro:property name="tyre_mass_ixx" value="2.53174430759784"/>
     <xacro:property name="tyre_mass_iyy" value="1.43724304615612"/>
@@ -94,5 +94,5 @@
     <xacro:property name="tyre_height" value="-0.696"/>
     <xacro:property name="str_mass" value="50.00"/>
-    <xacro:property name="str_length" value="0.01"/>
+    <xacro:property name="str_length" value="0.05"/>
     <xacro:property name="str_radius" value="0.1"/>
     <xacro:property name="front_right_offset" value="0.05"/>
@@ -279,5 +279,5 @@
         <parent link="base_link"/>
         <child link="front_right_steering_link"/>
-        <origin xyz="${tyre_front_x} ${-car_width/2 - str_length/2 + front_right_offset} ${tyre_r}" rpy="0 0 0"/>
+        <origin xyz="${tyre_front_x} ${-car_width/2 - 2*str_length} ${tyre_r}" rpy="0 0 0"/>
         <axis xyz="0 0 1"/>
         <limit effort="10000" lower="${-str_angle}" upper="${str_angle}" velocity="1000"/>
@@ -309,5 +309,5 @@
         <parent link="front_right_steering_link"/>
         <child link="front_right_wheel_link"/>
-        <origin xyz="0 ${-str_length/2 - tyre_length/2} 0" rpy="0 0 0"/>
+        <origin xyz="0 0 0" rpy="0 0 0"/>
         <axis xyz="0 1 0"/>
         <dynamics damping="0.01"/>
@@ -365,5 +365,5 @@
         <parent link="base_link"/>
         <child link="front_left_steering_link"/>
-        <origin xyz="${tyre_front_x} ${car_width/2 + str_length/2} ${tyre_r}" rpy="0 0 0"/>
+        <origin xyz="${tyre_front_x} ${car_width/2 + 2*str_length} ${tyre_r}" rpy="0 0 0"/>
         <axis xyz="0 0 1"/>
         <limit effort="10000" lower="${-str_angle}" upper="${str_angle}" velocity="1000"/>
@@ -396,5 +396,5 @@
           <parent link="front_left_steering_link"/>
           <child link="front_left_wheel_link"/>
-          <origin xyz="0 ${0.005 + tyre_length/2} 0" rpy="0 0 0"/>
+          <origin xyz="0 0 0" rpy="0 0 0"/>
           <axis xyz="0 1 0"/>
           <dynamics damping="0.01"/>

Commit message: Optional Obstaclestopper and sensor plugins, improved catvehicle tf

File: urdf/catvehicle.xacro (robot description, xacro)
@@ -33,5 +33,7 @@
     <xacro:arg name="triclops" default="true"/>
     <xacro:arg name="velodyne_points" default="true"/>
+    <xacro:arg name="laser_points" default="true"/>
     <xacro:property name="velodyne_points" value="$(arg velodyne_points)"/>
+    <xacro:property name="laser_points" value="$(arg laser_points)"/>
     <xacro:property name="camera_right" value="$(arg camera_right)"/>
     <xacro:property name="camera_left" value="$(arg camera_left)"/>
@@ -135,4 +137,7 @@
         <xacro:include filename="$(find catvehicle)/urdf/catvehicle_triclops.gazebo"/>
     </xacro:if>
+    <xacro:if value="${laser_points}">
+        <xacro:include filename="$(find catvehicle)/urdf/catvehicle_laser_points.gazebo"/>
+    </xacro:if>
     <!--Car Body-->
     <link name="base_link">
@@ -528,7 +533,6 @@
         </inertial>
     </link>
-    <!-- TRICLOPS -->
     <joint name="triclops" type="fixed">
-    <origin xyz="${sensor_box + camera_box/2} 0 ${0.725 + camera_box/2 + 1.25}" rpy="0 0 0"/>
+    <origin xyz="-0.25 0 ${0.725 + sensor_box/2 + 1.2}" rpy="0 0 0"/>
         <axis xyz="0 0 1"/>
         <parent link="base_link"/>
@@ -539,5 +543,5 @@
           <origin xyz="0 0 0" rpy="0 0 0"/>
           <geometry>
-           <box size="${camera_box/2} ${3*camera_box} ${camera_box/2}"/>
+          <box size="${camera_box/2} ${3*camera_box} ${camera_box/2}"/>
           </geometry>
         </collision>
@@ -554,33 +558,8 @@
         </inertial>
     </link>
-    <joint name="camera_joint" type="fixed">
-    <origin xyz="0 0 ${0.725 + sensor_box/2 + 1.25}" rpy="0 0 0"/>
-        <axis xyz="0 0 1"/>
-        <parent link="base_link"/>
-        <child link="camera_link"/>
-    </joint>
-    <link name="camera_link">
-        <collision>
-          <origin xyz="0 0 0" rpy="0 0 0"/>
-          <geometry>
-           <box size="${sensor_box} ${sensor_box} ${sensor_box}"/>
-          </geometry>
-        </collision>
-        <visual>
-          <origin xyz="0 0 0" rpy="0 0 0"/>
-          <geometry>
-          <box size="${sensor_box} ${sensor_box} ${sensor_box}"/>
-              </geometry>
-        </visual>
-        <inertial>
-          <mass value="1e-5" />
-          <origin xyz="0 0 0" rpy="0 0 0"/>
-          <inertia ixx="1e-6" ixy="0" ixz="0" iyy="1e-6" iyz="0" izz="1e-6" />
-        </inertial>
-    </link>
         <joint name="velodyne_joint" type="fixed">
-            <origin xyz="0 0 ${sensor_box/2 + 0.01}" rpy="0 0 0"/>
+            <origin xyz="-0.5 0 ${sensor_box/2 + 0.01}" rpy="0 0 0"/>
             <axis xyz="0 0 1"/>
-            <parent link="camera_link"/>
+            <parent link="triclops_link"/>
             <child link="velodyne_link"/>
         </joint>
